File: KiCad_PCB/PCB_Motor.kicad_pcb (KiCad board)
At the start: 4 copper layers, 100 x 100 mm, 33 parts, among them J2 Conn_01x02_Pin, U1 MOUDLE-SEEEDUINO-XIAO-ESP32C3, U2 LM321, U3 SS460S, U4 SS460S, U5 TMC6300, U6 SS460S

Commit message: Sync firmware and PCB
Routing:
- net (no net): track 0.00 -> 27641.9 mm, vias 0 -> 724
- net phase_a: track 9216.9 -> 0.00 mm, vias 240 -> 0
- net green: track 9213.8 -> 0.00 mm, vias 242 -> 0
- net blue: track 9211.3 -> 0.00 mm, vias 242 -> 0
- removed copper zone on B.Cu, net blue
- removed copper zone on B.Cu, net green
- removed copper zone on B.Cu, net phase_a
